File: PowerPlant-Module/PowerPlant-Module.kicad_pcb (KiCad board)
At the start: 4 copper layers, 22.5 x 37.7 mm, 35 parts, among them P2 CONN_01X02, P3 PWR, P4 CTRL, P5 LV_IO, P6 HV_IO, U4 LSF0204x, U5 LTC2942-1, U6 BQ24155, U7 SC283

Commit message: Silkscreen fix.
Other:
- board text added: "STAT ISEL REG_EN ~2V5 ~ALERT"
- board text removed: "REG_EN ~2V5 ISEL STAT ~ALERT"
Changed lines of the file:
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@@
-(kicad_pcb (version 4) (host pcbnew 4.0.4-stable)
+(kicad_pcb (version 4) (host pcbnew 4.0.6)
   (general
-    (links 0)
+    (links 123)
     (no_connects 0)
     (area -15.202501 15.795 58.072501 97.842101)
@@
     (34 B.Paste user)
     (35 F.Paste user)
-    (36 B.SilkS user hide)
+    (36 B.SilkS user)
     (37 F.SilkS user hide)
     (38 B.Mask user)
@@
   (gr_line (start 36.59 53.35) (end 36.59 45.984) (angle 90) (layer B.SilkS) (width 0.1))
   (gr_line (start 32.526 53.35) (end 36.59 53.35) (angle 90) (layer B.SilkS) (width 0.1))
-  (gr_text "BQ24155\nLTC2942-1\nSC283" (at 29.46 45.55 90) (layer B.Mask)
+  (gr_text "BQ24155\nLTC2942-1\nSC283" (at 29.65 45.55 90) (layer B.Mask)
     (effects (font (size 1 1) (thickness 0.18)) (justify left mirror))
   )
@@
     (effects (font (size 1.5 1.5) (thickness 0.2)) (justify left mirror))
   )
-  (gr_text "REG_EN\n~2V5\nISEL\nSTAT\n~ALERT" (at 19.064 47) (layer B.SilkS)
+  (gr_text "STAT\nISEL\nREG_EN\n~2V5\n~ALERT" (at 18.95 47.1) (layer B.SilkS)
     (effects (font (size 1.5 1.5) (thickness 0.2)) (justify right mirror))
   )
