File: r2-DevKit/r2-DevKit.sch (KiCad schematic (older format))
At the start: 29 parts, among them CON1 USB-MICRO-B, J1 CONN_01X05, J10 Battery SW, J11 OPTS, J2 CONN_01X08, J3 CONN_01X14, J4 CONN_01X02, J5 CONN_01X08, J6 CONN_01X14, J7 Li-Po, J8 JTAG, J9 CONN_02X15, P1 Compute Socket, P2 Sensor Socket, P3 CONN_01X01, P4 CONN_01X01, SW3 Pin_0, SW4 CHIP_PU, U1 EMIF02-USB03F2

Commit message: Adding BOM info.
Parts:
- D1, D2, D3: footprint Resistors_SMD:R_0402_NoSilk -> Diodes_SMD:D_0603; Digikey_Number LNJ347W83RACT-ND -> 732-4971-1-ND; Manu_Name Panasonic Electronic Components -> Wurth Electronics Inc.; Manu_Number LNJ347W83RA -> 150060GS75000
- J7: DigikeyNum 455-1749-6-ND -> (none); Digikey_Number (none) -> 455-1749-6-ND; ManuName JST Sales America Inc. -> (none); ManuNum S2B-PH-SM4-TB(LF)(SN) -> (none); Manu_Name (none) -> JST Sales America Inc.; Manu_Number (none) -> S2B-PH-SM4-TB(LF)(SN)
- R1, R4: Digikey_Number P1.00KLCT-ND -> 311-1.0KJRCT-ND; Manu_Name Panasonic Electronic Components -> Yageo; Manu_Number ERJ-2RKF1001X -> RC0402JR-071KL
- R2, R3: value 1k -> 680; Digikey_Number P1.00KLCT-ND -> 311-680JRCT-ND; Manu_Name Panasonic Electronic Components -> Yageo; Manu_Number ERJ-2RKF1001X -> RC0402JR-07680RL
Other:
- moved on the sheet: J8, P2, P3, P4

Commit message: Fixed some bugs in the Dev Harness.
Parts:
- removed J3, J6: CONN_01X14, Pin_Headers:Pin_Header_Straight_1x14_Pitch2.54mm, symbol CONN_01X14
- added CARY1, CARY2, CARY3: 100nF, r2Parts:CapArray_CKCL44, symbol CAPARRAY_4
- added J3: Conn_02x12_Odd_Even, Pin_Headers:Pin_Header_Straight_2x12_Pitch2.54mm, symbol Conn_02x12_Odd_Even
- added U2, U3, U4: LSF0204x, r2Parts:R-PUQFN-N12, symbol LSF0204x
- D1, D2, D3: footprint Diodes_SMD:D_0603 -> Resistors_SMD:R_0603_HandSoldering
- R1, R2, R3: footprint Resistors_SMD:R_0402_NoSilk -> Resistors_SMD:R_0603
- R4: footprint Resistors_SMD:R_0402_NoSilk -> Resistors_SMD:R_0603; Digikey_Number 311-1.0KJRCT-ND -> (none); Manu_Name Yageo -> (none); Manu_Number RC0402JR-071KL -> (none)
Connections:
- net CPLD_EXT_CLK: now also J3.20 (Pin_20)
- net CPLD_OE: now also J3.18 (Pin_18)
- net GND: now also J7.2 (P2), CARY1.2, CARY1.4, CARY1.6, CARY1.8, CARY2.2, CARY2.4, CARY2.6, CARY2.8, CARY3.2, CARY3.4, CARY3.6, CARY3.8, U2.6 (GND), U3.6 (GND), U4.6 (GND); no longer J7.1 (P1)
- net IRQ_WAKEUP: now also J3.2 (Pin_2)
- net SPI1_CLK: now also J3.8 (Pin_8)
- net SPI1_CS_0: now also J3.22 (Pin_22)
- net SPI1_MISO: now also J3.4 (Pin_4)
- net SPI1_MOSI: now also J3.6 (Pin_6)
- net SPI2_CLK: now also J3.14 (Pin_14)
- net SPI2_CS: now also J3.12 (Pin_12)
- net SPI2_MOSI: now also J3.10 (Pin_10)
- net VCC0: now also CARY1.5, CARY1.7, CARY2.5, CARY2.7, CARY3.5, CARY3.7, U2.11 (Vref_B), U3.11 (Vref_B), U4.11 (Vref_B)
- net VCC1: now also CARY1.1, CARY1.3, CARY2.1, CARY2.3, CARY3.1, CARY3.3, U2.1 (Vref_A), U3.1 (Vref_A), U4.1 (Vref_A)
- net ~CPLD_RESET: now also J3.16 (Pin_16)
- net ~REQ: now also J3.24 (Pin_24)
- net ~SHUTDOWN: now also U2.12 (EN), U3.12 (EN), U4.12 (EN)
- net at J10.1 (P1): now also J7.1 (P1); no longer J7.2 (P2)
- net at J9.10 (P10): now also U3.7 (B4)
- net at J9.8 (P8): now also U2.10 (B1)
- net at J9.6 (P6): now also U2.9 (B2)
- net at J9.4 (P4): now also U2.8 (B3)
- net at J9.2 (P2): now also U2.7 (B4)
- net at J9.24 (P24): now also U4.10 (B1)
- net at J9.22 (P22): now also U4.9 (B2)
- net at J9.20 (P20): now also U4.8 (B3)
- net at J9.18 (P18): now also U4.7 (B4)
- net at J9.16 (P16): now also U3.10 (B1)
- net at J9.14 (P14): now also U3.9 (B2)
- net at J9.12 (P12): now also U3.8 (B3)
- new net: J3.7 (Pin_7), U2.2 (A1)
- new net: J3.5 (Pin_5), U2.3 (A2)
- new net: J3.3 (Pin_3), U2.4 (A3)
- new net: J3.1 (Pin_1), U2.5 (A4)
- new net: J3.15 (Pin_15), U3.2 (A1)
- new net: J3.13 (Pin_13), U3.3 (A2)
- new net: J3.11 (Pin_11), U3.4 (A3)
- new net: J3.9 (Pin_9), U3.5 (A4)
- new net: J3.23 (Pin_23), U4.2 (A1)
- new net: J3.21 (Pin_21), U4.3 (A2)
- new net: J3.19 (Pin_19), U4.4 (A3)
- new net: J3.17 (Pin_17), U4.5 (A4)
Other:
- note removed: "Level-shifter socket"
- moved on the sheet: C1, CON1, D1, D2, D3, J1, J10, J11, J2, J4, J5, J7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
