File: Compute-WROOM32/Compute-WROOM32.sch (KiCad schematic (older format))
At the start: 15 parts, among them P1 HiRose-02X15, P4 CONN_01X01, U1 ESP32-WROOM, U2 FT231XS

Commit message: Filling in BOM.
Parts:
- C1: Digikey_Number (none) -> 399-1279-1-ND; Manu_Name (none) -> Kemet; Manu_Number (none) -> C0402C103J3RACTU
- C2: Digikey_Number (none) -> 478-8393-1-ND; Manu_Name (none) -> AVX Corporation; Manu_Number (none) -> F950J107MPAAQ2
- C3: Digikey_Number (none) -> 445-5947-1-ND; Manu_Name (none) -> TDK Corporation; Manu_Number (none) -> C1005X5R0J475K050BC
- C5, C6: Digikey_Number (none) -> 1276-1506-1-ND; Manu_Name (none) -> Samsung Electro-Mechanics America, Inc; Manu_Number (none) -> CL05B104JP5NNNC
- CARY1, CARY2, CARY3: Digikey_Number (none) -> 445-1838-1-ND; Manu_Name (none) -> TDK Corporation; Manu_Number (none) -> CKCL44X5R0J104M085AA
- CARY4: Digikey_Number 445-10063-1-ND -> 445-1824-1-ND; Manu_Number CKCA43CH1H220K100AA -> CKCL44C0G1H220K085AA
- P1: Digikey_Number (none) -> H5215CT-ND; Manu_Name (none) -> Hirose Electric Co Ltd; Manu_Number (none) -> DF12-30DS-0.5V(86)
- RP1: Digikey_Number (none) -> Y10153CT-ND; Manu_Name (none) -> Panasonic Electronic Components; Manu_Number (none) -> EXB-N8V153JX
- U1: Digikey_Number (none) -> 1528-1801-ND; Manu_Name (none) -> Espressif; Manu_Number (none) -> WROOM32
- U2: Digikey_Number (none) -> 768-1128-1-ND; Manu_Name (none) -> FTDI; Manu_Number (none) -> FT231XQ-R
Connections:
- no-connect marks 9 -> 19
Changed lines of the file:
@@
 LIBS:ESP32-footprints-Shem-Lib
 LIBS:IansParts
+LIBS:Compute-WROOM32-cache
 EELAYER 25 0
 EELAYER END
@@
 F 2 "ESP32-footprints-Lib:ESP32-WROOM" H 2850 5850 60  0001 C CNN
 F 3 "" H 2050 4950 60  0001 C CNN
+F 4 "WROOM32" H 2500 4500 60  0001 C CNN "Manu_Number"
+F 5 "Espressif" H 2500 4500 60  0001 C CNN "Manu_Name"
+F 6 "1528-1801-ND" H 2500 4500 60  0001 C CNN "Digikey_Number"
 	1    2500 4500
 	1    0    0    -1
@@
 F 2 "r2Parts:CapArray_CKCL44" H 5100 4400 60  0001 C CNN
 F 3 "" H 5100 4400 60  0000 C CNN
+F 4 "CKCL44X5R0J104M085AA" H 5100 4400 60  0001 C CNN "Manu_Number"
+F 5 "TDK Corporation" H 5100 4400 60  0001 C CNN "Manu_Name"
+F 6 "445-1838-1-ND" H 5100 4400 60  0001 C CNN "Digikey_Number"
 	1    5100 4400
 	0    -1   1    0
@@
 F 2 "r2Parts:CapArray_CKCL44" H 5100 3650 60  0001 C CNN
 F 3 "" H 5100 3650 60  0000 C CNN
+F 4 "CKCL44X5R0J104M085AA" H 5100 3650 60  0001 C CNN "Manu_Number"
+F 5 "TDK Corporation" H 5100 3650 60  0001 C CNN "Manu_Name"
+F 6 "445-1838-1-ND" H 5100 3650 60  0001 C CNN "Digikey_Number"
 	1    5100 3650
 	0    -1   1    0
@@
 F 2 "Capacitors_SMD:C_0402_NoSilk" H 5388 1000 50  0001 C CNN
 F 3 "" H 5350 1150 50  0000 C CNN
+F 4 "CL05B104JP5NNNC" H 5350 1150 60  0001 C CNN "Manu_Number"
+F 5 "Samsung Electro-Mechanics America, Inc" H 5350 1150 60  0001 C CNN "Manu_Name"
+F 6 "1276-1506-1-ND" H 5350 1150 60  0001 C CNN "Digikey_Number"
 	1    5350 1150
 	1    0    0    -1
@@
 F 2 "Capacitors_SMD:C_0402_NoSilk" H 4788 1000 50  0001 C CNN
 F 3 "" H 4750 1150 50  0000 C CNN
+F 4 "C1005X5R0J475K050BC" H 4750 1150 60  0001 C CNN "Manu_Number"
+F 5 "TDK Corporation" H 4750 1150 60  0001 C CNN "Manu_Name"
+F 6 "445-5947-1-ND" H 4750 1150 60  0001 C CNN "Digikey_Number"
 	1    4750 1150
 	1    0    0    -1
@@
 F 2 "Capacitors_SMD:C_0402_NoSilk" H 5038 1000 50  0001 C CNN
 F 3 "" H 5000 1150 50  0000 C CNN
+F 4 "CL05B104JP5NNNC" H 5000 1150 60  0001 C CNN "Manu_Number"
+F 5 "Samsung Electro-Mechanics America, Inc" H 5000 1150 60  0001 C CNN "Manu_Name"
+F 6 "1276-1506-1-ND" H 5000 1150 60  0001 C CNN "Digikey_Number"
 	1    5000 1150
 	1    0    0    -1
@@
 F 2 "Capacitors_SMD:C_0402_NoSilk" H 4538 1000 50  0001 C CNN
 F 3 "" H 4500 1150 50  0000 C CNN
+F 4 "C0402C103J3RACTU" H 4500 1150 60  0001 C CNN "Manu_Number"
+F 5 "Kemet" H 4500 1150 60  0001 C CNN "Manu_Name"
+F 6 "399-1279-1-ND" H 4500 1150 60  0001 C CNN "Digikey_Number"
 	1    4500 1150
 	1    0    0    -1
@@
 F 2 "r2Parts:CapArray_CKCL44" H 2650 1850 60  0001 C CNN
 F 3 "" H 2650 1850 60  0000 C CNN
+F 4 "CKCL44X5R0J104M085AA" H 2650 1850 60  0001 C CNN "Manu_Number"
+F 5 "TDK Corporation" H 2650 1850 60  0001 C CNN "Manu_Name"
+F 6 "445-1838-1-ND" H 2650 1850 60  0001 C CNN "Digikey_Number"
 	1    2650 1850
 	-1   0    0    -1
@@
 F 2 "r2Parts:RES_4_EXBN8V" V 2000 1150 50  0000 C CNN
 F 3 "" H 2350 1200 50  0000 C CNN
+F 4 "EXB-N8V153JX" H 2350 1200 60  0001 C CNN "Manu_Number"
+F 5 "Panasonic Electronic Components" H 2350 1200 60  0001 C CNN "Manu_Name"
+F 6 "Y10153CT-ND" H 2350 1200 60  0001 C CNN "Digikey_Number"
 	1    2350 1200
 	0    -1   1    0
@@
 F 2 "r2Parts:CapArray_CKCL44" H 5100 2550 60  0001 C CNN
 F 3 "" H 5100 2550 60  0000 C CNN
-F 4 "CKCA43CH1H220K100AA" H 5100 2550 60  0001 C CNN "Manu_Number"
+F 4 "CKCL44C0G1H220K085AA" H 5100 2550 60  0001 C CNN "Manu_Number"
 F 5 "TDK Corporation" H 5100 2550 60  0001 C CNN "Manu_Name"
-F 6 "445-10063-1-ND" H 5100 2550 60  0001 C CNN "Digikey_Number"
+F 6 "445-1824-1-ND" H 5100 2550 60  0001 C CNN "Digikey_Number"
 	1    5100 2550
 	0    -1   -1   0
@@
 F 2 "r2Parts:LFCSP_WQ20" H 6150 1800 60  0001 C CNN
 F 3 "" H 6150 1800 60  0001 C CNN
+F 4 "FT231XQ-R" V 6150 1800 60  0001 C CNN "Manu_Number"
+F 5 "FTDI" V 6150 1800 60  0001 C CNN "Manu_Name"
+F 6 "768-1128-1-ND" V 6150 1800 60  0001 C CNN "Digikey_Number"
 	1    6150 1800
 	1    0    0    -1
@@
 F 2 "r2Parts:DF12(4.0)-30DS-0.5V(86)" H 7950 2650 50  0000 C CNN
 F 3 "" H 7950 2650 50  0000 C CNN
+F 4 "DF12-30DS-0.5V(86)" H 7950 3800 60  0001 C CNN "Manu_Number"
+F 5 "Hirose Electric Co Ltd" H 7950 3800 60  0001 C CNN "Manu_Name"
+F 6 "H5215CT-ND" H 7950 3800 60  0001 C CNN "Digikey_Number"
 	1    7950 3800
 	-1   0    0    -1
@@
 F 2 "Capacitors_SMD:C_0805" H 6050 3700 60  0001 C CNN
 F 3 "" H 6050 3700 60  0000 C CNN
+F 4 "F950J107MPAAQ2" V 6050 3700 60  0001 C CNN "Manu_Number"
+F 5 "AVX Corporation" V 6050 3700 60  0001 C CNN "Manu_Name"
+F 6 "478-8393-1-ND" V 6050 3700 60  0001 C CNN "Digikey_Number"
 	1    6050 3700
 	1    0    0    -1
@@
 Text Label 7650 3100 2    39   ~ 0
 CHIP_PU
+NoConn ~ 2100 1400
+NoConn ~ 2000 1400
+NoConn ~ 1550 4200
+NoConn ~ 1550 4100
+NoConn ~ 2250 5550
+NoConn ~ 2350 5550
+NoConn ~ 2450 5550
+NoConn ~ 2550 5550
+NoConn ~ 2650 5550
+NoConn ~ 2750 5550
 $EndSCHEMATC

Commit message: Updated compute module to fix a bug, and to use the WROOM32-U.
Parts:
- removed CARY2: 100nF, r2Parts:CapArray_CKCL44, symbol CAPARRAY_4
- removed U1: ESP32-WROOM, ESP32-footprints-Lib:ESP32-WROOM, symbol ESP32-WROOM
- added U1: ESP32-WROOM_U, ESP32-footprints-Lib:ESP32-WROOM-U, symbol ESP32-footprints-Shem-Lib:ESP32-WROOM_U
- C1, C3, C5, C6: symbol C -> Compute-WROOM32-rescue:C
- C2: symbol IANS_CAP_POLARIZED -> IansParts:IANS_CAP_POLARIZED
- CARY1, CARY3, CARY4: symbol CAPARRAY_4 -> IansParts:CAPARRAY_4
- P1: symbol HiRose-02X15 -> IansParts:HiRose-02X15
- P4: symbol CONN_01X01 -> Compute-WROOM32-rescue:CONN_01X01
- QA_NPN1: symbol QA_NPN -> IansParts:QA_NPN
- RP1: symbol R_PACK4 -> Compute-WROOM32-rescue:R_PACK4
- U2: symbol FT231XS -> IansParts:FT231XS
Connections:
- wire segments 152 -> 176
- no-connect marks 19 -> 20

Commit message: Updating to r2 backplane fixes from last year.
Changed lines of the file:
@@
 Text Label 1500 3800 2    39   ~ 0
 CHIP_PU
-Text Label 1500 4500 2    39   ~ 0
+Text Label 1500 4800 2    39   ~ 0
 SPI1_MOSI
 Text Label 3450 4800 0    39   ~ 0
 CPLD_OE
-Text Label 1500 4800 2    39   ~ 0
+Text Label 1500 4500 2    39   ~ 0
 SPI1_MISO
 Text Label 3450 4400 0    39   ~ 0

Commit message: Compute module will now take either WROOM32 module.
Parts:
- added RP2: 15k, r2Parts:RES_4_EXBN8V, symbol Compute-WROOM32-rescue:R_PACK4
- added U3: ASTMLP, r2Parts:ASTMLPD, symbol IansParts:ASTMLP
Connections:
- wire segments 176 -> 191
- no-connect marks 20 -> 22
Changed lines of the file:
@@
 Text Label 1500 4300 2    39   ~ 0
 IRQ_WAKEUP
-Text Label 3450 4700 0    39   ~ 0
+Text Label 4900 4300 0    39   ~ 0
 CPLD_EXT_CLK
 Text Label 1500 4200 2    39   ~ 0
@@
 	3400 4800 3450 4800
 Wire Wire Line
-	3400 4700 3450 4700
-Wire Wire Line
 	3450 4500 3400 4500
 Wire Wire Line
@@
 	1500 3800 1550 3800
 NoConn ~ 2850 5350
+$Comp
+L Compute-WROOM32-rescue:R_PACK4 RP2
+U 1 1 5C52DC57
+P 5600 4900
+F 0 "RP2" H 5600 5350 50  0000 C CNN
+F 1 "15k" H 5600 4850 50  0000 C CNN
+F 2 "r2Parts:RES_4_EXBN8V" H 5500 4750 50  0000 C CNN
+F 3 "" H 5600 4900 50  0000 C CNN
+F 4 "EXB-38V102JV" H 5600 4900 60  0001 C CNN "Manu_Number"
+F 5 "Panasonic Electronic Components" H 5600 4900 60  0001 C CNN "Manu_Name"
+F 6 "Y9102CT-ND" H 5600 4900 60  0001 C CNN "Digikey_Number"
+	1    5600 4900
+	-1   0    0    -1
+$EndComp
+Text Label 5350 4750 2    39   ~ 0
+I2C_SDA
+Text Label 5350 4850 2    39   ~ 0
+I2C_SCL
+Wire Wire Line
+	5350 4850 5400 4850
+Wire Wire Line
+	5400 4750 5350 4750
+Wire Wire Line
+	5800 4850 5850 4850
+Wire Wire Line
+	5850 4850 5850 4750
+Wire Wire Line
+	5850 4550 5800 4550
+Wire Wire Line
+	5800 4650 5850 4650
+Connection ~ 5850 4650
+Wire Wire Line
+	5850 4650 5850 4550
+Wire Wire Line
+	5800 4750 5850 4750
+Connection ~ 5850 4750
+Wire Wire Line
+	5850 4750 5850 4650
+Text Label 5950 4650 0    39   ~ 0
+VCC0
+Wire Wire Line
+	5950 4650 5850 4650
+NoConn ~ 5400 4650
+NoConn ~ 5400 4550
+$Comp
+L IansParts:ASTMLP U3
+U 1 1 5C599D6C
+P 4450 4400
+F 0 "U3" H 4500 4725 50  0000 C CNN
+F 1 "ASTMLP" H 4500 4634 50  0000 C CNN
+F 2 "r2Parts:ASTMLPD" H 4450 4400 50  0001 C CNN
+F 3 "" H 4450 4400 50  0001 C CNN
+F 4 "ASTMLPD-16.000MHZ-LJ-E-T‎" H 4450 4400 50  0001 C CNN "Manu_Number"
+F 5 "Abracon" H 4450 4400 50  0001 C CNN "Manu_Name"
+F 6 "‎535-13087-1-ND‎" H 4450 4400 50  0001 C CNN "Digikey_Number"
+	1    4450 4400
+	1    0    0    -1
+$EndComp
+Text Label 4100 4450 2    39   ~ 0
+GND
+Wire Wire Line
+	4100 4450 4150 4450
+Wire Wire Line
+	4850 4300 4900 4300
+Text Label 4900 4450 0    39   ~ 0
+VCC0
+Wire Wire Line
+	4900 4450 4850 4450
+Wire Wire Line
+	3850 4700 3850 4300
+Wire Wire Line
+	3850 4300 4150 4300
+Wire Wire Line
+	3400 4700 3850 4700
 $EndSCHEMATC
