File: r2-Backplane/r2-Backplane.sch (KiCad schematic (older format))
At the start: 44 parts, among them CON1 USB-MICRO-B, P1 CONN_01X01, P2 CONN_01X02, P3 CONN_02X16, P4 HiRose-02X15, P6 DEBUG, U1 LSF0204x, U2 LSF0204x, U3 LSF0204x, U4 LSF0204x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

Commit message: BOM filled out, but board not verified.
Parts:
- removed L3: 2.2uH, r2Parts:L-SMD, symbol L_Core_Ferrite
- removed R2, R5, R6: 10k, Resistors_SMD:R_0402_NoSilk, symbol R
- added L2: 2.2uH, r2Parts:L-SMD, symbol L_Core_Ferrite
- added RP2: 10k, r2Parts:RES_4_EXBN8V, symbol R_Pack04
- C1, C3, C7: Digikey_Number (none) -> 490-1320-1-ND; Manu_Name (none) -> Murata Electronics North America; Manu_Number (none) -> GRM155R60J105KE19D
- C10, C5: Digikey_Number (none) -> 490-3340-1-ND; Manu_Name (none) -> Murata Electronics North America; Manu_Number (none) -> GRM219R60J106KE19D
- C11, C4: Digikey_Number (none) -> 490-1719-1-ND; Manu_Name (none) -> Murata Electronics North America; Manu_Number (none) -> GRM21BR60J226ME39L
- C12: Digikey_Number (none) -> 1276-1506-1-ND; Manu_Name (none) -> Samsung Electro-Mechanics America, Inc; Manu_Number (none) -> CL05B104JP5NNNC
- C2: Digikey_Number (none) -> 490-3335-1-ND; Manu_Name (none) -> Murata Electronics North America; Manu_Number (none) -> GRM21BR61E475KA12L
- C6, C9: Digikey_Number (none) -> 490-3340-1-ND; Manu_Name (none) -> Murata Electronics North America; Manu_Number (none) -> 490-3340-1-ND
- C8: Digikey_Number (none) -> 399-1279-1-ND; Manu_Name (none) -> Kemet; Manu_Number (none) -> C0402C103J3RACTU
- D1: Digikey_Number (none) -> LNJ347W83RACT-ND; Manu_Name (none) -> Panasonic Electronic Components; Manu_Number (none) -> LNJ347W83RA
- F1: Digikey_Number (none) -> NANOSMDC075F-2CT-ND; Manu_Name (none) -> Littelfuse Inc.; Manu_Number (none) -> NANOSMDC075F-2
- L1: Digikey_Number (none) -> 308-2294-1-ND; Manu_Name (none) -> Sumida America Components Inc.; Manu_Number (none) -> CDRH2D14NP-2R2NC
- L3: footprint r2Parts:L-SMD -> Inductors_NEOSID:Neosid_Inductor_SM-NE29_SMD1008
- P4: Manu_Name (none) -> Hirose Electric Co Ltd; Manu_Number (none) -> DF12(4.0)-30DP-0.5V(86)
- R1: Digikey_Number (none) -> P1.00KLCT-ND; Manu_Name (none) -> Panasonic Electronic Components; Manu_Number (none) -> ERJ-2RKF1001X
- R3: value 470 -> 1k; Digikey_Number (none) -> P1.00KLCT-ND; Manu_Name (none) -> Panasonic Electronic Components; Manu_Number (none) -> ERJ-2RKF1001X
- R4: Digikey_Number (none) -> CSRN2512FK68L0CT-ND; Manu_Name (none) -> Stackpole Electronics Inc.; Manu_Number (none) -> CSRN2512FK68L0
- RP1: Digikey_Number (none) -> Y10220CT-ND; Manu_Name (none) -> Panasonic Electronic Components; Manu_Number (none) -> EXB-N8V220JX
- U1, U2, U3, U4: Digikey_Number (none) -> 296-40404-1-ND; Manu_Name (none) -> Texas Instruments; Manu_Number (none) -> LSF0204RUTR
- U6: Digikey_Number (none) -> 296-27187-1-ND; Manu_Name (none) -> Texas Instruments; Manu_Number (none) -> BQ24155RGYR
- U7: Digikey_Number (none) -> SC283WLCT-ND; Manu_Name (none) -> Semtech Corporation; Manu_Number (none) -> SC283WLTRT
- U8: Digikey_Number (none) -> 497-13521-1-ND; Manu_Name (none) -> STMicroelectronics; Manu_Number (none) -> EMIF02-USB03F2
Connections:
- wire segments 297 -> 299
- no-connect marks 11 -> 12
Other:
- note removed: "NOTE: This is actually an NC7SV57."
- moved on the sheet: R1, RP1

Commit message: Adding small tools catch-all project.
Connections:
- wire segments 299 -> 307
- no-connect marks 12 -> 7

Commit message: Adding modules.
Parts:
- P3: Digikey_Number H5205CT-ND -> H11708TR-ND
Changed lines of the file:
@@
 F 4 "DF12-32DS-0.5V(86)" H 10150 4150 39  0001 C CNN "Manu_Number"
 F 5 "Hirose Electric Co Ltd" H 10150 5000 39  0001 C CNN "Manu_Name"
-F 6 "H5205CT-ND" H 10150 5000 39  0001 C CNN "Digikey_Number"
+F 6 "H11708TR-ND" H 10150 5000 39  0001 C CNN "Digikey_Number"
 	1    10150 5000
 	-1   0    0    1

Commit message: Updating to r2 backplane fixes from last year.
Parts:
- C1, C10, C11, C12, C2, C3, C4, C5, C6, C7, C8, C9: symbol C -> r2-Backplane-rescue:C
- CARY1, CARY2, CARY3, CARY4, CARY5: symbol CAPARRAY_4 -> IansParts:CAPARRAY_4
- CON1: symbol USB-MICRO-B -> IansParts:USB-MICRO-B
- D1: symbol LED_Small -> r2-Backplane-rescue:LED_Small
- F1: symbol Polyfuse_Small -> r2-Backplane-rescue:Polyfuse_Small
- L1, L2, L3: symbol L_Core_Ferrite -> r2-Backplane-rescue:L_Core_Ferrite
- P1: symbol CONN_01X01 -> r2-Backplane-rescue:CONN_01X01
- P2: symbol CONN_01X02 -> r2-Backplane-rescue:CONN_01X02
- P3: symbol CONN_02X16 -> r2-Backplane-rescue:CONN_02X16
- P4: symbol HiRose-02X15 -> IansParts:HiRose-02X15
- P6: symbol CONN_01X08 -> r2-Backplane-rescue:CONN_01X08
- QA_NPN1: symbol QA_NPN -> IansParts:QA_NPN
- R1, R3, R4: symbol R -> r2-Backplane-rescue:R
- RP1, RP2: symbol R_Pack04 -> r2-Backplane-rescue:R_Pack04
- U1, U2, U3, U4: symbol LSF0204x -> IansParts:LSF0204x
- U5: symbol LTC2942 -> IansParts:LTC2942
- U6: symbol BQ24155 -> IansParts:BQ24155
- U7: symbol SC283 -> IansParts:SC283
- U8: symbol EMIF02-USB03F2 -> IansParts:EMIF02-USB03F2
Connections:
- wire segments 307 -> 394

Commit message: Compute module will now take either WROOM32 module.
Parts:
- RP2: value 10k -> 1k; Digikey_Number Y10103CT-ND -> Y9102CT-ND; Manu_Number EXB-N8V103JX -> EXB-38V102JV
Changed lines of the file:
@@
 P 6900 2050
 F 0 "RP2" V 6600 2050 50  0000 C CNN
-F 1 "10k" V 7100 2050 50  0000 C CNN
+F 1 "1k" V 7100 2050 50  0000 C CNN
 F 2 "r2Parts:RES_4_EXBN8V" V 7175 2050 50  0001 C CNN
 F 3 "" H 6900 2050 50  0001 C CNN
-F 4 "EXB-N8V103JX" V 6900 2050 60  0001 C CNN "Manu_Number"
+F 4 "EXB-38V102JV" V 6900 2050 60  0001 C CNN "Manu_Number"
 F 5 "Panasonic Electronic Components" V 6900 2050 60  0001 C CNN "Manu_Name"
-F 6 "Y10103CT-ND" V 6900 2050 60  0001 C CNN "Digikey_Number"
+F 6 "Y9102CT-ND" V 6900 2050 60  0001 C CNN "Digikey_Number"
 	1    6900 2050
 	0    1    1    0
